Commit message: Add color detection and point cloud analysis.

File: turtlebot3/turtlebot3_description/urdf/turtlebot3_burger.gazebo.xacro (robot description, xacro)
@@ -124,3 +124,44 @@
     </sensor>
   </gazebo>
+  <gazebo reference="camera_link">
+    <sensor name="camera" type="depth">
+      <update_rate>20</update_rate>
+      <camera>
+      <horizontal_fov>1.047198</horizontal_fov>
+      <image>
+          <width>640</width>
+          <height>480</height>
+          <format>R8G8B8</format>
+      </image>
+      <clip>
+          <near>0.05</near>
+          <far>30</far>
+      </clip>
+      </camera>
+      <plugin name="camera_plugin" filename="libgazebo_ros_openni_kinect.so">
+      <baseline>0.2</baseline>
+      <alwaysOn>true</alwaysOn>
+      <updateRate>0.0</updateRate>
+      <cameraName>camera_ir</cameraName>
+      <imageTopicName>/camera/color/image_raw</imageTopicName>
+      <cameraInfoTopicName>/camera/color/camera_info</cameraInfoTopicName>
+      <depthImageTopicName>/camera/depth/image_raw</depthImageTopicName>
+      <depthImageCameraInfoTopicName>/camera/depth/camera_info</depthImageCameraInfoTopicName>
+      <pointCloudTopicName>/camera/depth/points</pointCloudTopicName>
+      <frameName>camera_link</frameName>
+      <pointCloudCutoff>0.5</pointCloudCutoff>
+      <pointCloudCutoffMax>30.0</pointCloudCutoffMax>
+      <distortionK1>0</distortionK1>
+      <distortionK2>0</distortionK2>
+      <distortionK3>0</distortionK3>
+      <distortionT1>0</distortionT1>
+      <distortionT2>0</distortionT2>
+      <CxPrime>0</CxPrime>
+      <Cx>0</Cx>
+      <Cy>0</Cy>
+      <focalLength>0</focalLength>
+      <hackBaseline>0</hackBaseline>
+      </plugin>
+    </sensor>
+  </gazebo>
 </robot>

File: turtlebot3/turtlebot3_description/urdf/turtlebot3_burger.urdf.xacro (robot description, xacro)
@@ -140,3 +140,10 @@
     </inertial>
   </link>
+  <!-- Add camera -->
+  <joint name="camera_joint" type="fixed">
+      <origin rpy="0 0 0" xyz="0 0 0.5" />
+      <parent link="base_link" />
+      <child link="camera_link" />
+  </joint>
+  <link name="camera_link" />
 </robot>
